Commit message: joitn5 and link6 remove

File: indy-ros2/indy_description/urdf/indy.ros2_control.xacro (robot description, xacro)
@@ -44,8 +44,8 @@
             <xacro:define_control_joint joint_index="joint3"/>
             <xacro:define_control_joint joint_index="joint4"/>
-            <xacro:define_control_joint joint_index="joint5"/>
+            <!-- <xacro:define_control_joint joint_index="joint5"/>
             <xacro:if value="${indy_type == 'indyrp2' or indy_type == 'indyrp2_v2'}">
                 <xacro:define_control_joint joint_index="joint6"/>
-            </xacro:if>
+            </xacro:if> -->
         </ros2_control>
     </xacro:macro>

File: indy-ros2/indy_description/urdf/indy_macro.xacro (robot description, xacro)
@@ -66,8 +66,8 @@
         <xacro:define_link link_index="link5" link_mesh="link5"/>
         <xacro:if value="${indy_eye and not (indy_type == 'indyrp2' or indy_type == 'indyrp2_v2')}">
-            <xacro:define_link link_index="link6" link_mesh="link6_eye"/>
+            <!-- <xacro:define_link link_index="link6" link_mesh="link6_eye"/> -->
         </xacro:if>
         <xacro:unless value="${indy_eye and not (indy_type == 'indyrp2' or indy_type == 'indyrp2_v2')}">
-            <xacro:define_link link_index="link6" link_mesh="link6"/>
+            <!-- <xacro:define_link link_index="link6" link_mesh="link6"/> -->
         </xacro:unless>
         <xacro:if value="${indy_type == 'indyrp2' or indy_type == 'indyrp2_v2'}">
@@ -114,5 +114,5 @@
         <xacro:define_joint joint_index="joint3" link_1_index="link3" link_2_index="link4"/>
         <xacro:define_joint joint_index="joint4" link_1_index="link4" link_2_index="link5"/>
-        <xacro:define_joint joint_index="joint5" link_1_index="link5" link_2_index="link6"/>
+        <!-- <xacro:define_joint joint_index="joint5" link_1_index="link5" link_2_index="link6"/> -->
         <xacro:if value="${indy_type == 'indyrp2' or indy_type == 'indyrp2_v2'}">
             <xacro:define_joint joint_index="joint6" link_1_index="link6" link_2_index="link7"/>
@@ -125,7 +125,7 @@
         <xacro:unless value="${indy_type == 'indyrp2' or indy_type == 'indyrp2_v2'}">
             <joint name="${prefix}tcp" type="fixed">
-                <parent link="${prefix}link6"/>
+                <parent link="${prefix}link5"/>
                 <child link="${prefix}tcp"/>
-                <origin xyz="0 0 0.06" rpy="0 0 0"/>
+                <origin xyz="0 0 0.1" rpy="0 0 0"/>
             </joint>
         </xacro:unless>

File: indy-ros2/indy_description/urdf/indy_transmissions.xacro (robot description, xacro)
@@ -18,5 +18,5 @@
         <xacro:define_transmission tran="tran3" joint="joint3" motor="motor3"/>
         <xacro:define_transmission tran="tran4" joint="joint4" motor="motor4"/>
-        <xacro:define_transmission tran="tran5" joint="joint5" motor="motor5"/>
+        <!-- <xacro:define_transmission tran="tran5" joint="joint5" motor="motor5"/> -->
         <!--indyrp2 with 7 DOF-->
         <xacro:if value="${indy_type == 'indyrp2' or indy_type == 'indyrp2_v2'}">

File: indy-ros2/indy_moveit/srdf/indy_macro.srdf.xacro (robot description, xacro)
@@ -54,5 +54,5 @@
                 <joint name="${prefix}joint3" value="0" />
                 <joint name="${prefix}joint4" value="0" />
-                <joint name="${prefix}joint5" value="0" />
+                <!-- <joint name="${prefix}joint5" value="0" /> -->
             </group_state>
             <group_state name="${prefix}ZeroPos" group="${prefix}${name}_manipulator">
@@ -62,5 +62,5 @@
                 <joint name="${prefix}joint3" value="0" />
                 <joint name="${prefix}joint4" value="0" />
-                <joint name="${prefix}joint5" value="0" />
+                <!-- <joint name="${prefix}joint5" value="0" /> -->
             </group_state>
             <!--END EFFECTOR - Purpose - Represent information about an end effector.-->
@@ -73,5 +73,5 @@
             <disable_collisions link1="link3" link2="link4" reason="Adjacent" />
             <disable_collisions link1="link4" link2="link5" reason="Adjacent" />
-            <disable_collisions link1="link5" link2="link6" reason="Adjacent" />
+            <!-- <disable_collisions link1="link5" link2="link6" reason="Adjacent" /> -->
             <disable_collisions link1="link2" link2="link4" reason="Never" />
             <disable_collisions link1="link2" link2="link5" reason="Never" />
@@ -79,5 +79,5 @@
             <disable_collisions link1="link3" link2="link5" reason="Never" />
             <disable_collisions link1="link3" link2="link6" reason="Never" />
-            <disable_collisions link1="link4" link2="link6" reason="Never" />
+            <!-- <disable_collisions link1="link4" link2="link6" reason="Never" /> -->
         </xacro:unless>
     </xacro:macro>
