Commit message: setting change

File: indy-ros2/indy_description/urdf/indy_macro.xacro (robot description, xacro)
@@ -127,5 +127,5 @@
                 <parent link="${prefix}link5"/>
                 <child link="${prefix}tcp"/>
-                <origin xyz="0 0 0.1" rpy="0 0 0"/>
+                <origin xyz="0 0.5 0" rpy="0 0 0"/>
             </joint>
         </xacro:unless>

Commit message: link6 changed grip position because link6's joint limit disturbs planning

File: indy-ros2/indy_description/urdf/indy_macro.xacro (robot description, xacro)
@@ -127,5 +127,5 @@
                 <parent link="${prefix}link6"/>
                 <child link="${prefix}tcp"/>
-                <origin xyz="0 0 0.06" rpy="0 0 0"/>
+                <origin xyz="0 0 0" rpy="0 0 0"/>
             </joint>
         </xacro:unless>

Commit message: poseset command added.

File: indy-ros2/indy_description/urdf/indy_macro.xacro (robot description, xacro)
@@ -66,5 +66,29 @@
         <xacro:define_link link_index="link5" link_mesh="link5"/>
         <xacro:if value="${indy_eye and not (indy_type == 'indyrp2' or indy_type == 'indyrp2_v2')}">
-            <xacro:define_link link_index="link6" link_mesh="link6_eye"/>
+            <joint name="camera_joint" type="fixed">
+		<parent link="link0"/>
+		<child link="camera_link"/>
+		<origin xyz="-0.123 -0.13 0.7" rpy="0 1.0996 -1.57075"/>
+	    </joint>
+	    <xacro:define_link link_index="camera_link" link_mesh=""/>
+	    <link name="camera_link">
+		<visual>
+		    <geometry>
+			<mesh filename="package://urdfbot_description/meshes/visual/mani_camera.stl" scale="0.001 0.001 0.001"/>
+		    </geometry>
+		</visual>
+		<collision>
+		    <geometry>
+			<mesh filename="package://urdfbot_description/meshes/visual/mani_camera.stl" scale="0.001 0.001 0.001"/>
+		    </geometry>
+		</collision>
+	    </link>
+	    <joint name="camera_optical_joint" type="fixed">
+		<parent link="camera_link"/>
+		<child link="camera_link_optical"/>
+		<origin xyz="0 0 0" rpy="-1.57075 0 -1.57075"/>
+	    </joint>
+	    <link name="camera_link_optical">
+	    </link>
         </xacro:if>
         <xacro:unless value="${indy_eye and not (indy_type == 'indyrp2' or indy_type == 'indyrp2_v2')}">

File: indy-ros2/indy_moveit/srdf/indy_macro.srdf.xacro (robot description, xacro)
@@ -18,9 +18,9 @@
             <group_state name="${prefix}HomePos" group="${prefix}${name}_manipulator">
                 <joint name="${prefix}joint0" value="0" />
-                <joint name="${prefix}joint1" value="0" />
-                <joint name="${prefix}joint2" value="0" />
-                <joint name="${prefix}joint3" value="-1.570796327" />
-                <joint name="${prefix}joint4" value="0" />
-                <joint name="${prefix}joint5" value="-1.570796327" />
+                <joint name="${prefix}joint1" value="1.4312" />
+                <joint name="${prefix}joint2" value="-1.5359" />
+                <joint name="${prefix}joint3" value="0" />
+                <joint name="${prefix}joint4" value="-0.1745" />
+                <joint name="${prefix}joint5" value="0" />
                 <joint name="${prefix}joint6" value="0" />
             </group_state>
@@ -50,8 +50,8 @@
             <group_state name="${prefix}HomePos" group="${prefix}${name}_manipulator">
                 <joint name="${prefix}joint0" value="0" />
-                <joint name="${prefix}joint1" value="0" />
-                <joint name="${prefix}joint2" value="-1.570796327" />
+                <joint name="${prefix}joint1" value="1.4312" />
+                <joint name="${prefix}joint2" value="-1.5359" />
                 <joint name="${prefix}joint3" value="0" />
-                <joint name="${prefix}joint4" value="-1.570796327" />
+                <joint name="${prefix}joint4" value="-0.1745" />
                 <joint name="${prefix}joint5" value="0" />
             </group_state>
@@ -68,4 +68,8 @@
             <virtual_joint name="FixedBase" type="fixed" parent_frame="global" child_link="world" />
             <!--DISABLE COLLISIONS - By default it is assumed that any link of the robot could potentially come into collision with any other link in the robot. This tag disables collision checking between a specified pair of links. -->
+            <disable_collisions link1="camera_link" link2="link0" reason="Adjacent"/>
+    	    <disable_collisions link1="camera_link" link2="link1" reason="Never"/>
+    	    <disable_collisions link1="camera_link" link2="link2" reason="Never"/>
+    	    <disable_collisions link1="camera_link" link2="link3" reason="Never"/>
             <disable_collisions link1="link0" link2="link1" reason="Adjacent" />
             <disable_collisions link1="link1" link2="link2" reason="Adjacent" />

File: urdfbot_description/urdf/urdfbot_simple.urdf (robot description, URDF)
Before this commit: robot urdfbot, 8 links, 7 joints
Links:
- added link camera_link; collision mesh filename=package://urdfbot_description/meshes/visual/mani_camera.stl scale=0.001 0.001 0.001; visual mesh filename=package://urdfbot_description/meshes/visual/mani_camera.stl scale=0.001 0.001 0.001
- added link camera_link_optical
Joints:
- added joint camera_joint: type fixed, parent mani_link1, child camera_link, origin xyz=-0.123 -0.13 0.7 rpy=0 1.0996 -1.57075
- added joint camera_optical_joint: type fixed, parent camera_link, child camera_link_optical, origin xyz=0 0 0 rpy=-1.57075 0 -1.57075
