Commit message: mani urdf package

File: urdfbot_description/urdf/urdfbot_simple.urdf (robot description, URDF)
Before this commit: robot urdfbot, 7 links, 6 joints
Links:
- link mani_link1: geometry collision mesh filename=package://urdfbot_description/meshes/collision/mani_1.stl scale=0.001 0.001 0.001; visual mesh filename=package://urdfbot_description/meshes/visual/mani_1.stl scale=0.001 0.001 0.001
- link mani_link2: geometry collision mesh filename=package://urdfbot_description/meshes/collision/mani_2.stl scale=0.001 0.001 0.001; visual mesh filename=package://urdfbot_description/meshes/visual/mani_2.stl scale=0.001 0.001 0.001
- link mani_link3: geometry collision mesh filename=package://urdfbot_description/meshes/collision/mani_3.stl scale=0.001 0.001 0.001; visual mesh filename=package://urdfbot_description/meshes/visual/mani_3.stl scale=0.001 0.001 0.001
- link mani_link4: geometry collision mesh filename=package://urdfbot_description/meshes/collision/mani_4.stl scale=0.001 0.001 0.001; visual mesh filename=package://urdfbot_description/meshes/visual/mani_4.stl scale=0.001 0.001 0.001
- link mani_link5: geometry collision mesh filename=package://urdfbot_description/meshes/collision/mani_5.stl scale=0.001 0.001 0.001; visual mesh filename=package://urdfbot_description/meshes/visual/mani_5.stl scale=0.001 0.001 0.001
- link mani_link6: geometry collision mesh filename=package://urdfbot_description/meshes/collision/mani_6.stl scale=0.001 0.001 0.001; visual mesh filename=package://urdfbot_description/meshes/visual/mani_6.stl scale=0.001 0.001 0.001
- link mani_link7: geometry collision mesh filename=package://urdfbot_description/meshes/collision/mani_7.stl scale=0.001 0.001 0.001; visual mesh filename=package://urdfbot_description/meshes/visual/mani_7.stl scale=0.001 0.001 0.001
Joints:
- joint mani_joint1: origin xyz=0 0 62 rpy=0 0 0 -> xyz=0 0 0.062 rpy=0 0 0
- joint mani_joint2: limit lower=-2.9671 upper=2.9671 effort=87 velocity=2.3925 -> lower=-1.57075 upper=1.57075 effort=87 velocity=2.3925; origin xyz=22.85 0 47 rpy=0 -1.57075 0 -> xyz=0.02285 0 0.047 rpy=0 -1.57075 0
- joint mani_joint3: limit lower=-2.9671 upper=2.9671 effort=87 velocity=2.3925 -> lower=-1.57075 upper=1.57075 effort=87 velocity=2.3925; origin xyz=319.5 0 45.5 rpy=0 0 1.57075 -> xyz=0.3195 0 0.0455 rpy=0 0 0
- joint mani_joint4: origin xyz=66.0 -64 -22 rpy=0 -1.57075 1.57075 -> xyz=0.066 -0.064 -0.022 rpy=0 -1.57075 1.57075
- joint mani_joint5: axis 0 0 1 -> 1 0 0; limit lower=-2.9671 upper=2.9671 effort=87 velocity=2.3925 -> lower=-1.57075 upper=1.57075 effort=87 velocity=2.3925; origin xyz=0 0 248.75 rpy=0 0 0 -> xyz=0 0 0.24875 rpy=0 0 0
- joint mani_joint6: origin xyz=0 0 56.5 rpy=0 0 0 -> xyz=0 0 0.0565 rpy=0 0 0

Commit message: moveit with 8th virtual link

File: urdfbot_description/urdf/urdfbot_simple.urdf (robot description, URDF)
Before this commit: robot urdfbot, 7 links, 6 joints
Links:
- added link mani_link8; visual sphere radius=0.001
Joints:
- added joint mani_joint7: type revolute, parent mani_link7, child mani_link8, origin xyz=0 0 0.110 rpy=0 0 0, axis 1 0 0, limit lower=-3.1415 upper=3.1415 effort=87 velocity=2.3925

Commit message: manipulator coordinate control complete + dynamixel pub

File: urdfbot_description/urdf/urdfbot_simple.urdf (robot description, URDF)
Before this commit: robot urdfbot, 8 links, 7 joints
Links:
- added link camera_link; collision box size=0.01 0.03 0.03; visual box size=0.01 0.03 0.03
- added link camera_link_optical
Joints:
- added joint camera_joint: type fixed, parent mani_link5, child camera_link, origin xyz=0 -0.03 0.23 rpy=0 -1.57075 0
- added joint camera_optical_joint: type fixed, parent camera_link, child camera_link_optical, origin xyz=0 0 0 rpy=-1.57075 0 -1.57075

Commit message: mani stl change

File: urdfbot_description/urdf/urdfbot_simple.urdf (robot description, URDF)
Before this commit: robot urdfbot, 8 links, 7 joints
Joints:
- joint mani_joint1: origin xyz=0 0 0.062 rpy=0 0 0 -> xyz=0 0 0.073 rpy=0 0 0
- joint mani_joint2: origin xyz=0.02285 0 0.047 rpy=0 -1.57075 0 -> xyz=0.02285 0 0.051 rpy=0 -1.57075 0

Commit message: joystick + real robot complete

File: urdfbot_description/urdf/urdfbot_simple.urdf (robot description, URDF)
Before this commit: robot urdfbot, 8 links, 7 joints
Joints:
- joint mani_joint1: origin xyz=0 0 0.073 rpy=0 0 0 -> xyz=0 0 0.103 rpy=0 0 0
