Commit message: home position set

File: indy-ros2/indy_moveit/srdf/indy_macro.srdf.xacro (robot description, xacro)
@@ -18,15 +18,15 @@
             <group_state name="${prefix}HomePos" group="${prefix}${name}_manipulator">
                 <joint name="${prefix}joint0" value="0" />
-                <joint name="${prefix}joint1" value="0" />
-                <joint name="${prefix}joint2" value="0" />
-                <joint name="${prefix}joint3" value="-1.570796327" />
+                <joint name="${prefix}joint1" value="0.872665" />
+                <joint name="${prefix}joint2" value="-0.872665" />
+                <joint name="${prefix}joint3" value="0" />
                 <joint name="${prefix}joint4" value="0" />
-                <joint name="${prefix}joint5" value="-1.570796327" />
+                <joint name="${prefix}joint5" value="0" />
                 <joint name="${prefix}joint6" value="0" />
             </group_state>
             <group_state name="${prefix}ZeroPos" group="${prefix}${name}_manipulator">
                 <joint name="${prefix}joint0" value="0" />
-                <joint name="${prefix}joint1" value="0" />
-                <joint name="${prefix}joint2" value="0" />
+                <joint name="${prefix}joint1" value="0.872665" />
+                <joint name="${prefix}joint2" value="-0.872665" />
                 <joint name="${prefix}joint3" value="0" />
                 <joint name="${prefix}joint4" value="0" />

Commit message: subscriber finish

File: indy-ros2/indy_moveit/srdf/indy_macro.srdf.xacro (robot description, xacro)
@@ -27,6 +27,6 @@
             <group_state name="${prefix}ZeroPos" group="${prefix}${name}_manipulator">
                 <joint name="${prefix}joint0" value="0" />
-                <joint name="${prefix}joint1" value="0.872665" />
-                <joint name="${prefix}joint2" value="-0.872665" />
+                <joint name="${prefix}joint1" value="1.570796327" />
+                <joint name="${prefix}joint2" value="-1.570796327" />
                 <joint name="${prefix}joint3" value="0" />
                 <joint name="${prefix}joint4" value="0" />
@@ -50,14 +50,14 @@
             <group_state name="${prefix}HomePos" group="${prefix}${name}_manipulator">
                 <joint name="${prefix}joint0" value="0" />
-                <joint name="${prefix}joint1" value="0" />
-                <joint name="${prefix}joint2" value="-1.570796327" />
+                <joint name="${prefix}joint1" value="0.872665" />
+                <joint name="${prefix}joint2" value="-0.872665" />
                 <joint name="${prefix}joint3" value="0" />
-                <joint name="${prefix}joint4" value="-1.570796327" />
+                <joint name="${prefix}joint4" value="0" />
                 <joint name="${prefix}joint5" value="0" />
             </group_state>
             <group_state name="${prefix}ZeroPos" group="${prefix}${name}_manipulator">
                 <joint name="${prefix}joint0" value="0" />
-                <joint name="${prefix}joint1" value="0" />
-                <joint name="${prefix}joint2" value="0" />
+                <joint name="${prefix}joint1" value="1.570796327" />
+                <joint name="${prefix}joint2" value="-1.570796327" />
                 <joint name="${prefix}joint3" value="0" />
                 <joint name="${prefix}joint4" value="0" />

Commit message: homepos joint4 change

File: indy-ros2/indy_moveit/srdf/indy_macro.srdf.xacro (robot description, xacro)
@@ -21,5 +21,5 @@
                 <joint name="${prefix}joint2" value="-1.5359" />
                 <joint name="${prefix}joint3" value="0" />
-                <joint name="${prefix}joint4" value="-0.1745" />
+                <joint name="${prefix}joint4" value="0" />
                 <joint name="${prefix}joint5" value="0" />
                 <joint name="${prefix}joint6" value="0" />

Commit message: homepos joint4 change

File: indy-ros2/indy_moveit/srdf/indy_macro.srdf.xacro (robot description, xacro)
@@ -21,5 +21,5 @@
                 <joint name="${prefix}joint2" value="-1.5359" />
                 <joint name="${prefix}joint3" value="0" />
-                <joint name="${prefix}joint4" value="0" />
+                <joint name="${prefix}joint4" value="1.57075" />
                 <joint name="${prefix}joint5" value="0" />
                 <joint name="${prefix}joint6" value="0" />
@@ -53,5 +53,5 @@
                 <joint name="${prefix}joint2" value="-1.5359" />
                 <joint name="${prefix}joint3" value="0" />
-                <joint name="${prefix}joint4" value="-0.1745" />
+                <joint name="${prefix}joint4" value="1.57075" />
                 <joint name="${prefix}joint5" value="0" />
             </group_state>

Commit message: upload backup

File: indy-ros2/indy_moveit/srdf/indy_macro.srdf.xacro (robot description, xacro)
@@ -31,4 +31,13 @@
                 <joint name="${prefix}joint3" value="0" />
                 <joint name="${prefix}joint4" value="0" />
+                <joint name="${prefix}joint5" value="0" />
+                <joint name="${prefix}joint6" value="0" />
+            </group_state>
+            <group_state name="${prefix}ServoPos" group="${prefix}${name}_manipulator">
+                <joint name="${prefix}joint0" value="0" />
+                <joint name="${prefix}joint1" value="-0.2443" />
+                <joint name="${prefix}joint2" value="-0.3141" />
+                <joint name="${prefix}joint3" value="0" />
+                <joint name="${prefix}joint4" value="-0.9075" />
                 <joint name="${prefix}joint5" value="0" />
                 <joint name="${prefix}joint6" value="0" />
